Commit message: simplified robot with gripper

File: robot_description/xarm_description/xarm6/urdf/xarm6_with_gripper.urdf (robot description, URDF)
Before this commit: robot xarm6_with_gripper, 15 links, 14 joints
Links:
- link left_finger: geometry collision mesh filename=package://xarm6/meshes/xarm_gripper/left_finger.obj; visual mesh filename=package://xarm6/meshes/xarm_gripper/left_finger.obj
- link left_inner_knuckle: geometry collision mesh filename=package://xarm6/meshes/xarm_gripper/left_inner_knuckle.obj; visual mesh filename=package://xarm6/meshes/xarm_gripper/left_inner_knuckle.obj
- link left_outer_knuckle: geometry collision mesh filename=package://xarm6/meshes/xarm_gripper/left_outer_knuckle.obj; visual mesh filename=package://xarm6/meshes/xarm_gripper/left_outer_knuckle.obj
- link link1: geometry collision mesh filename=package://xarm6/meshes/xarm6/collision/link1.obj; visual mesh filename=package://xarm6/meshes/xarm6/visual/link1.obj
- link link2: geometry collision mesh filename=package://xarm6/meshes/xarm6/collision/link2.obj; visual mesh filename=package://xarm6/meshes/xarm6/visual/link2.obj
- link link3: geometry collision mesh filename=package://xarm6/meshes/xarm6/collision/link3.obj; visual mesh filename=package://xarm6/meshes/xarm6/visual/link3.obj
- link link4: geometry collision mesh filename=package://xarm6/meshes/xarm6/collision/link4.obj; visual mesh filename=package://xarm6/meshes/xarm6/visual/link4.obj
- link link5: geometry collision mesh filename=package://xarm6/meshes/xarm6/collision/link5.obj; visual mesh filename=package://xarm6/meshes/xarm6/visual/link5.obj
- link link6: geometry collision mesh filename=package://xarm6/meshes/xarm6/visual/link6.obj; visual mesh filename=package://xarm6/meshes/xarm6/visual/link6.obj
- link link_base: geometry collision mesh filename=package://xarm6/meshes/xarm6/collision/base.obj; visual mesh filename=package://xarm6/meshes/xarm6/visual/base.obj
- link right_finger: geometry collision mesh filename=package://xarm6/meshes/xarm_gripper/right_finger.obj; visual mesh filename=package://xarm6/meshes/xarm_gripper/right_finger.obj
- link right_inner_knuckle: geometry collision mesh filename=package://xarm6/meshes/xarm_gripper/right_inner_knuckle.obj; visual mesh filename=package://xarm6/meshes/xarm_gripper/right_inner_knuckle.obj
- link right_outer_knuckle: geometry collision mesh filename=package://xarm6/meshes/xarm_gripper/right_outer_knuckle.obj; visual mesh filename=package://xarm6/meshes/xarm_gripper/right_outer_knuckle.obj
- link xarm_gripper_base_link: geometry collision mesh filename=package://xarm6/meshes/xarm_gripper/base_link.obj; visual mesh filename=package://xarm6/meshes/xarm_gripper/base_link.obj

File: robot_description/xarm_description/xarm6/urdf/xarm6_with_parallel_gripper.urdf (robot description, URDF)
Before this commit: robot xarm6_with_gripper, 15 links, 14 joints
Links:
- link left_finger: geometry collision mesh filename=package://xarm6/meshes/xarm_gripper/left_finger.obj; visual mesh filename=package://xarm6/meshes/xarm_gripper/left_finger.obj
- link left_inner_knuckle: geometry collision mesh filename=package://xarm6/meshes/xarm_gripper/left_inner_knuckle.obj; visual mesh filename=package://xarm6/meshes/xarm_gripper/left_inner_knuckle.obj
- link left_outer_knuckle: geometry collision mesh filename=package://xarm6/meshes/xarm_gripper/left_outer_knuckle.obj; visual mesh filename=package://xarm6/meshes/xarm_gripper/left_outer_knuckle.obj
- link link1: geometry collision mesh filename=package://xarm6/meshes/xarm6/collision/link1.obj; visual mesh filename=package://xarm6/meshes/xarm6/visual/link1.obj
- link link2: geometry collision mesh filename=package://xarm6/meshes/xarm6/collision/link2.obj; visual mesh filename=package://xarm6/meshes/xarm6/visual/link2.obj
- link link3: geometry collision mesh filename=package://xarm6/meshes/xarm6/collision/link3.obj; visual mesh filename=package://xarm6/meshes/xarm6/visual/link3.obj
- link link4: geometry collision mesh filename=package://xarm6/meshes/xarm6/collision/link4.obj; visual mesh filename=package://xarm6/meshes/xarm6/visual/link4.obj
- link link5: geometry collision mesh filename=package://xarm6/meshes/xarm6/collision/link5.obj; visual mesh filename=package://xarm6/meshes/xarm6/visual/link5.obj
- link link6: geometry collision mesh filename=package://xarm6/meshes/xarm6/visual/link6.obj; visual mesh filename=package://xarm6/meshes/xarm6/visual/link6.obj
- link link_base: geometry collision mesh filename=package://xarm6/meshes/xarm6/collision/base.obj; visual mesh filename=package://xarm6/meshes/xarm6/visual/base.obj
- link right_finger: geometry collision mesh filename=package://xarm6/meshes/xarm_gripper/right_finger.obj; visual mesh filename=package://xarm6/meshes/xarm_gripper/right_finger.obj
- link right_inner_knuckle: geometry collision mesh filename=package://xarm6/meshes/xarm_gripper/right_inner_knuckle.obj; visual mesh filename=package://xarm6/meshes/xarm_gripper/right_inner_knuckle.obj
- link right_outer_knuckle: geometry collision mesh filename=package://xarm6/meshes/xarm_gripper/right_outer_knuckle.obj; visual mesh filename=package://xarm6/meshes/xarm_gripper/right_outer_knuckle.obj
- link xarm_gripper_base_link: geometry collision mesh filename=package://xarm6/meshes/xarm_gripper/base_link.obj; visual mesh filename=package://xarm6/meshes/xarm_gripper/base_link.obj
Joints:
- joint drive_joint: axis 1 0 0 -> (none); limit lower=0 upper=0.85 effort=50 velocity=2 -> (none); type revolute -> fixed
- joint left_finger_joint: axis -1 0 0 -> 0 1 0; limit lower=0 upper=0.85 effort=50 velocity=2 -> lower=-0.045 upper=0 effort=50 velocity=2; mimic joint=drive_joint multiplier=1 offset=0 -> (none); origin xyz=0 0.035465 0.042039 rpy=0 0 0 -> xyz=0 0.070465 0.101137 rpy=0 0 0; parent left_outer_knuckle -> xarm_gripper_base_link; type revolute -> prismatic
- joint left_inner_knuckle_joint: axis 1 0 0 -> (none); limit lower=0 upper=0.85 effort=50 velocity=2 -> (none); mimic joint=drive_joint multiplier=1 offset=0 -> (none); type revolute -> fixed
- joint right_finger_joint: axis 1 0 0 -> 0 -1 0; limit lower=0 upper=0.85 effort=50 velocity=2 -> lower=-0.045 upper=0 effort=50 velocity=2; mimic joint=drive_joint multiplier=1 offset=0 -> (none); origin xyz=0 -0.035465 0.042039 rpy=0 0 0 -> xyz=0 -0.070465 0.101137 rpy=0 0 0; parent right_outer_knuckle -> xarm_gripper_base_link; type revolute -> prismatic
- joint right_inner_knuckle_joint: axis -1 0 0 -> (none); limit lower=0 upper=0.85 effort=50 velocity=2 -> (none); mimic joint=drive_joint multiplier=1 offset=0 -> (none); type revolute -> fixed
- joint right_outer_knuckle_joint: axis -1 0 0 -> (none); limit lower=0 upper=0.85 effort=50 velocity=2 -> (none); mimic joint=drive_joint multiplier=1 offset=0 -> (none); type revolute -> fixed
