Commit message: scara env

File: robot_description/scara/urdf/scara.urdf (robot description, URDF)
Before this commit: robot robot-assembly-2, 3 links, 2 joints
Links:
- link base_link: geometry collision mesh filename=package://scara/meshes/base_link.STL; visual mesh filename=package://scara/meshes/base_link.STL
- link link_1: geometry collision mesh filename=package://scara/meshes/link_1.STL; visual mesh filename=package://scara/meshes/link_1.STL
- link link_2: geometry collision mesh filename=package://scara/meshes/link_2.STL; visual mesh filename=package://scara/meshes/link_2.STL
