Commit message: can move scara splat

File: robot_description/scara_25-04-08/urdf/scara.urdf (robot description, URDF)
Before this commit: robot scara, 4 links, 3 joints
Links:
- removed link link_3
- added link gripper, mass 0.007854; collision mesh filename=package://scara/meshes/gripper.STL; visual mesh filename=package://scara/meshes/gripper.STL
Joints:
- removed joint joint_1
- removed joint joint_2
- removed joint joint_3
- added joint elbow: type revolute, parent link_1, child link_2, origin xyz=0.15462 0.05041 0.13618 rpy=-0.015862 0.97874 -0.030813, axis 0 1 0, limit lower=0 upper=0 effort=0 velocity=0
- added joint gripper_linear: type prismatic, parent link_2, child gripper, origin xyz=0.094697 0 -0.16386 rpy=1.5708 1.5021 0, axis 0 0 1, limit lower=0 upper=0 effort=0 velocity=0
- added joint shoulder: type revolute, parent base_link, child link_1, origin xyz=0 0 0 rpy=1.5708 0 -0.44269, axis 0 1 0, limit lower=0 upper=0 effort=0 velocity=0
